Commit message: remove uwb

File: models/husky/urdf/ugv.urdf.xacro (robot description, xacro)
@@ -2,183 +2,21 @@
 <robot name="husky" xmlns:xacro="http://ros.org/wiki/xacro">
   <xacro:include filename="$(find husky_description)/urdf/husky.urdf.xacro" />
-  <link name="platform_link">
+  <link name="marker_link">
     <visual>
       <cast_shadows>true</cast_shadows>
       <geometry>
-        <mesh filename="package://mp_uav_landing_sim/models/husky/meshes/platform.dae" scale="0.5 0.5 0.5"/>
+        <mesh filename="package://uav_landing/models/husky/meshes/marker.dae" />
       </geometry>
     </visual>
     <collision>
       <geometry>
-        <mesh filename="package://mp_uav_landing_sim/models/husky/meshes/platform.dae" scale="0.5 0.5 0.5"/>
-      </geometry>
-    </collision>
-  </link>
-  <joint name="platform_joint" type="fixed">
-    <parent link="base_link" />
-    <child link="platform_link" />
-    <origin xyz="-0.02 0 0.36" rpy="0 0 3.14" />
-  </joint>
-  <link name="anchor0_link">
-    <visual>
-      <cast_shadows>true</cast_shadows>
-      <geometry>
-        <mesh filename="package://mp_uav_landing_sim/models/husky/meshes/uwb_anchor.dae" scale="1 1 1"/>
-      </geometry>
-    </visual>
-    <collision>
-      <geometry>
-        <mesh filename="package://mp_uav_landing_sim/models/husky/meshes/uwb_anchor.dae" scale="1 1 1"/>
-      </geometry>
-    </collision>
-  </link>
-  <joint name="anchor0_joint" type="fixed">
-    <parent link="platform_link" />
-    <child link="anchor0_link" />
-    <origin xyz="-0.67 -0.518 0.09" rpy="0 0 1.57" />
-  </joint>
-  <link name="anchor1_link">
-    <visual>
-      <cast_shadows>true</cast_shadows>
-      <geometry>
-        <mesh filename="package://mp_uav_landing_sim/models/husky/meshes/uwb_anchor.dae" scale="1 1 1"/>
-      </geometry>
-    </visual>
-    <collision>
-      <geometry>
-        <mesh filename="package://mp_uav_landing_sim/models/husky/meshes/uwb_anchor.dae" scale="1 1 1"/>
-      </geometry>
-    </collision>
-  </link>
-  <joint name="anchor1_joint" type="fixed">
-    <parent link="platform_link" />
-    <child link="anchor1_link" />
-    <origin xyz="-0.67 0.55 0.06" rpy="0 0 1.57" />
-  </joint>
-  <link name="anchor2_link">
-    <visual>
-      <cast_shadows>true</cast_shadows>
-      <geometry>
-        <mesh filename="package://mp_uav_landing_sim/models/husky/meshes/uwb_anchor.dae" scale="1 1 1"/>
-      </geometry>
-    </visual>
-    <collision>
-      <geometry>
-        <mesh filename="package://mp_uav_landing_sim/models/husky/meshes/uwb_anchor.dae" scale="1 1 1"/>
-      </geometry>
-    </collision>
-  </link>
-  <joint name="anchor2_joint" type="fixed">
-    <parent link="platform_link" />
-    <child link="anchor2_link" />
-    <origin xyz="0.57 -0.518 0.09" rpy="0 0 1.57" />
-  </joint>
-  <link name="anchor3_link">
-    <visual>
-      <cast_shadows>true</cast_shadows>
-      <geometry>
-        <mesh filename="package://mp_uav_landing_sim/models/husky/meshes/uwb_anchor.dae" scale="1 1 1"/>
-      </geometry>
-    </visual>
-    <collision>
-      <geometry>
-        <mesh filename="package://mp_uav_landing_sim/models/husky/meshes/uwb_anchor.dae" scale="1 1 1"/>
-      </geometry>
-    </collision>
-  </link>
-  <joint name="anchor3_joint" type="fixed">
-    <parent link="platform_link" />
-    <child link="anchor3_link" />
-    <origin xyz="0.57 0.55 0.09" rpy="0 0 1.57" />
-  </joint>
-    <link name="marker_link">
-    <visual>
-      <cast_shadows>true</cast_shadows>
-      <geometry>
-        <mesh filename="package://mp_uav_landing_sim/models/husky/meshes/marker.dae" />
-      </geometry>
-    </visual>
-    <collision>
-      <geometry>
-        <mesh filename="package://mp_uav_landing_sim/models/husky/meshes/marker.dae" />
+        <mesh filename="package://uav_landing/models/husky/meshes/marker.dae" />
       </geometry>
     </collision>
   </link>
   <joint name="marker_joint" type="fixed">
-    <parent link="platform_link" />
+    <parent link="base_link" />
     <child link="marker_link" />
-    <origin xyz="-0.05 0 0.02" rpy="0 0 0" />
-  </joint>
-  <link name="diode0_link">
-    <visual>
-      <cast_shadows>true</cast_shadows>
-      <geometry>
-        <mesh filename="package://mp_uav_landing_sim/models/husky/meshes/diode.dae" scale="0.4 0.4 0.4"/>
-      </geometry>
-    </visual>
-    <collision>
-      <geometry>
-        <mesh filename="package://mp_uav_landing_sim/models/husky/meshes/diode.dae" scale="0.4 0.4 0.4"/>
-      </geometry>
-    </collision>
-  </link>
-  <joint name="diode0_joint" type="fixed">
-    <parent link="platform_link" />
-    <child link="diode0_link" />
-    <origin xyz="-0.85 0.42 0.64" rpy="0 0 0" />
-  </joint>
-  <link name="diode1_link">
-    <visual>
-      <cast_shadows>true</cast_shadows>
-      <geometry>
-        <mesh filename="package://mp_uav_landing_sim/models/husky/meshes/diode.dae" scale="0.4 0.4 0.4"/>
-      </geometry>
-    </visual>
-    <collision>
-      <geometry>
-        <mesh filename="package://mp_uav_landing_sim/models/husky/meshes/diode.dae" scale="0.4 0.4 0.4"/>
-      </geometry>
-    </collision>
-  </link>
-  <joint name="diode1_joint" type="fixed">
-    <parent link="platform_link" />
-    <child link="diode1_link" />
-    <origin xyz="-0.85 -0.45 0.64" rpy="0 0 0" />
-  </joint>
-  <link name="diode2_link">
-    <visual>
-      <cast_shadows>true</cast_shadows>
-      <geometry>
-        <mesh filename="package://mp_uav_landing_sim/models/husky/meshes/diode.dae" scale="0.4 0.4 0.4"/>
-      </geometry>
-    </visual>
-    <collision>
-      <geometry>
-        <mesh filename="package://mp_uav_landing_sim/models/husky/meshes/diode.dae" scale="0.4 0.4 0.4"/>
-      </geometry>
-    </collision>
-  </link>
-  <joint name="diode2_joint" type="fixed">
-    <parent link="platform_link" />
-    <child link="diode2_link" />
-    <origin xyz="-0.85 -0.01 1" rpy="1.57 0 0" />
-  </joint>
-  <link name="diode3_link">
-    <visual>
-      <cast_shadows>true</cast_shadows>
-      <geometry>
-        <mesh filename="package://mp_uav_landing_sim/models/husky/meshes/diode.dae" scale="0.4 0.4 0.4"/>
-      </geometry>
-    </visual>
-    <collision>
-      <geometry>
-        <mesh filename="package://mp_uav_landing_sim/models/husky/meshes/diode.dae" scale="0.4 0.4 0.4"/>
-      </geometry>
-    </collision>
-  </link>
-  <joint name="diode3_joint" type="fixed">
-    <parent link="platform_link" />
-    <child link="diode3_link" />
-    <origin xyz="-0.85 -0.01 0.2" rpy="1.57 0 0" />
+    <origin xyz="-0.02 0 0.36" rpy="0 0 0" />
   </joint>
 </robot>
